Commit message: The urdf has been spawned properly need to add the gazebo part for the movement

File: mapping_robot/urdf/mapping_robot.urdf (robot description, URDF)
Before this commit: robot mapping_robot, 3 links, 2 joints
Joints:
- joint left_wheel_joint: origin xyz=0.37685 -0.26212 -0.4793 rpy=0 0 0 -> xyz=0.0 0 0 rpy=0 0 0
- joint right_wheel_joint: origin xyz=0.49222 0.21894 -0.47244 rpy=1.5708 0 0 -> xyz=0.0 0.0 0.0 rpy=1.5708 0 0

File: mapping_robot_1/urdf/mapping_robot_1.urdf (robot description, URDF)
Before this commit: robot mapping_robot_`1, 3 links, 2 joints
Links:
- link Left_link: geometry collision mesh filename=package://mapping_robot_1/meshes/Left_link.STL; visual mesh filename=package://mapping_robot_1/meshes/Left_link.STL
- link Right_Link: geometry collision mesh filename=package://mapping_robot_1/meshes/Right_Link.STL; visual mesh filename=package://mapping_robot_1/meshes/Right_Link.STL
- link base_link: geometry collision mesh filename=package://mapping_robot_1/meshes/base_link.STL; visual mesh filename=package://mapping_robot_1/meshes/base_link.STL
Joints:
- joint Right_wheel: limit lower=0 upper=0 effort=0 velocity=0 -> lower=0 upper=6.28 effort=0 velocity=0; origin xyz=-0.010873 0.009058 -0.0074666 rpy=0 0 0 -> xyz=-0.07 0.0 -0.005 rpy=0 0 0
- joint left_wheel: limit lower=0 upper=0 effort=0 velocity=0 -> lower=0 upper=6.28 effort=0 velocity=0; origin xyz=0 0 0 rpy=0 0 0 -> xyz=0.07 0.0 -0.005 rpy=0 0 0
