Commit message: Added camera plugins and the robot can rotate in place

File: mapping_robot_1/urdf/mapping_robot_1.urdf (robot description, URDF)
Before this commit: robot mapping_robot_1, 3 links, 2 joints
Links:
- added link camera_link; collision box size=0.003975 0.00795 0.007155
- added link camera_link1; collision box size=0.003975 0.00795 0.007155
- added link camera_rgb_frame
- added link camera_rgb_frame1
- added link camera_rgb_optical_frame
- added link camera_rgb_optical_frame1
- link base_link: geometry collision mesh filename=package://mapping_robot_1/meshes/base_link.STL; collision sphere radius=0.015
Joints:
- added joint camera_joint: type fixed, parent base_link, child camera_link, origin xyz=0.015 0.05 0.2 rpy=0 0 1.57
- added joint camera_joint1: type fixed, parent base_link, child camera_link1, origin xyz=-0.015 0.05 0.2 rpy=0 0 1.57
- added joint camera_rgb_joint: type fixed, parent camera_link, child camera_rgb_frame, origin xyz=0.000795 0.002915 0.002385 rpy=0 0 0
- added joint camera_rgb_joint1: type fixed, parent camera_link1, child camera_rgb_frame1, origin xyz=0.000795 0.002915 0.002385 rpy=0 0 0
- added joint camera_rgb_optical_joint: type fixed, parent camera_rgb_frame, child camera_rgb_optical_frame, origin xyz=0 0 0 rpy=-1.57 0 -1.57
- added joint camera_rgb_optical_joint1: type fixed, parent camera_rgb_frame1, child camera_rgb_optical_frame1, origin xyz=0 0 0 rpy=-1.57 0 -1.57
- joint Right_wheel: limit lower=0 upper=6.28 effort=0 velocity=0 -> effort=20 velocity=10; origin xyz=-0.07 0.0 -0.005 rpy=0 0 0 -> xyz=-0.07 0.0 -0.009 rpy=0 0 0; type revolute -> continuous
- joint left_wheel: axis 1 0 0 -> -1 0 0; limit lower=0 upper=6.28 effort=0 velocity=0 -> effort=20 velocity=10; origin xyz=0.07 0.0 -0.005 rpy=0 0 0 -> xyz=0.07 0.0 -0.009 rpy=0 0 0; type revolute -> continuous

Commit message: added the camera and the stereo link

File: mapping_robot_1/urdf/mapping_robot_1.urdf (robot description, URDF)
Before this commit: robot mapping_robot_1, 9 links, 8 joints
Links:
- added link caster_front; collision sphere radius=0.015; visual sphere radius=0.015
- added link caster_front1; collision sphere radius=0.015; visual sphere radius=0.015
- added link stereo_link; collision box size=0.007 0.035 0.01; visual box size=0.007 0.035 0.01
- link base_link: geometry collision mesh filename=package://mapping_robot_1/meshes/base_link.STL; visual mesh filename=package://mapping_robot_1/meshes/base_link.STL
Joints:
- added joint caster_joint: type fixed, parent base_link, child caster_front, origin xyz=0 0.08 -0.02 rpy=0 0 0
- added joint caster_joint1: type fixed, parent base_link, child caster_front1, origin xyz=0 -0.08 -0.02 rpy=0 0 0
- added joint stereo_joint: type fixed, parent base_link, child stereo_link, origin xyz=0.0 0.065 0.21 rpy=0 0 1.57
- joint camera_joint: origin xyz=0.015 0.05 0.2 rpy=0 0 1.57 -> xyz=0.0165 0.065 0.21 rpy=0 0 1.57
- joint camera_joint1: origin xyz=-0.015 0.05 0.2 rpy=0 0 1.57 -> xyz=-0.0135 0.065 0.21 rpy=0 0 1.57
